File: v1.0/thingBot-Base_v1P0.kicad_pcb (KiCad board)
At the start: 2 copper layers, 45 x 53 mm, 113 parts, among them P1 MICRO_USB, P2 BATT_CONN, P3 XBEE_CONN_LEFT, P4 CONN_01X02, P5 CONN_01X02, P6 JTAG, P7 XBEE, P8 XBEE_CONN_RIGHT, SW1 ON/OFF_Switch, U2 CP2102, U3 LP5907_LDO_250mA, U4 PROBE

Commit message: final Layout and GERBER creation done
Parts:
- removed the REF** at (160.7, 113.0)
- removed the REF** at (144.7, 119.0)
- removed the REF** at (155.8, 100.2)
- removed the REF** at (155.8, 98.2)
- removed the REF** at (155.8, 96.2)
- removed the REF** at (155.8, 94.2)
- removed the REF** at (155.8, 92.2)
- removed the REF** at (155.8, 90.2)
- removed the REF** at (155.8, 88.2)
- removed the REF** at (155.8, 86.2)
- removed the REF** at (155.8, 84.2)
- removed the REF** at (155.8, 82.2)
- removed the REF** at (155.8, 80.2)
- removed the REF** at (164.6, 125.7)
- removed the REF** at (133.8, 110.2)
- removed the REF** at (133.8, 108.2)
- removed the REF** at (133.8, 106.2)
- removed the REF** at (133.8, 104.2)
- removed the REF** at (133.8, 102.2)
- removed the REF** at (133.8, 100.2)
- removed the REF** at (133.8, 98.2)
- removed the REF** at (133.8, 96.2)
- removed the REF** at (133.8, 94.2)
- removed the REF** at (133.8, 92.2)
- removed the REF** at (133.8, 90.2)
- removed the REF** at (133.8, 88.2)
- removed the REF** at (133.8, 86.2)
- removed the REF** at (152.6, 113.4)
- removed the REF** at (133.8, 84.2)
- removed the REF** at (133.8, 82.2)
- removed the REF** at (133.8, 80.2)
- removed the REF** at (175.8, 114.2)
- removed the REF** at (175.8, 112.2)
- removed the REF** at (175.8, 110.2)
- removed the REF** at (175.8, 108.2)
- removed the REF** at (175.8, 106.2)
- removed the REF** at (175.8, 104.2)
- removed the REF** at (175.8, 102.2)
- removed the REF** at (146.7, 123.0)
- removed the REF** at (175.8, 100.2)
- removed the REF** at (175.8, 98.2)
- removed the REF** at (175.8, 96.2)
- removed the REF** at (175.8, 94.2)
- removed the REF** at (175.8, 92.2)
- removed the REF** at (175.8, 90.2)
- removed the REF** at (175.8, 88.2)
- removed the REF** at (175.8, 86.2)
- removed the REF** at (175.8, 84.2)
- removed the REF** at (175.8, 82.2)
- removed the REF** at (144.7, 123.0)
- removed the REF** at (175.8, 80.2)
- removed the REF** at (173.8, 78.2)
- removed the REF** at (171.8, 78.2)
- removed the REF** at (169.8, 78.2)
- removed the REF** at (167.8, 78.2)
- removed the REF** at (165.8, 78.2)
- removed the REF** at (163.8, 78.2)
- removed the REF** at (161.8, 78.2)
- removed the REF** at (159.8, 78.2)
- removed the REF** at (157.8, 78.2)
- removed the REF** at (146.7, 121.0)
- removed the REF** at (153.8, 78.2)
- removed the REF** at (151.8, 78.2)
- removed the REF** at (149.8, 78.2)
- removed the REF** at (147.8, 78.2)
- removed the REF** at (145.8, 78.2)
- removed the REF** at (143.8, 78.2)
- removed the REF** at (141.8, 78.2)
- removed the REF** at (139.8, 78.2)
- removed the REF** at (137.8, 78.2)
- removed the REF** at (144.7, 121.0)
- removed the REF** at (135.8, 78.2)
- removed the REF** at (141.4, 126.4)
- removed the REF** at (164.6, 121.7)
- removed the REF** at (135.0, 128.8)
- removed the REF** at (139.2, 124.0)
- removed the REF** at (146.7, 119.0)
- added REF**: VAL**, conn-wire-pads:Hole-Screw-NP-#4, F.Cu at (128.3, 71.6)
- added REF**: VIA_0.6mm, VIA'S:VIA_0.6mm, F.Cu at (127.7, 90.8)
- added REF**: VIA_0.6mm, VIA'S:VIA_0.6mm, F.Cu at (127.7, 85.8)
- added REF**: VIA_0.6mm, VIA'S:VIA_0.6mm, F.Cu at (127.7, 80.8)
- added REF**: VIA_0.6mm, VIA'S:VIA_0.6mm, F.Cu at (127.7, 75.8)
- added REF**: VIA_0.6mm, VIA'S:VIA_0.6mm, F.Cu at (169.8, 105.8)
- added REF**: VIA_0.6mm, VIA'S:VIA_0.6mm, F.Cu at (169.8, 95.8)
- added REF**: VIA_0.6mm, VIA'S:VIA_0.6mm, F.Cu at (169.8, 90.8)
- added REF**: VIA_0.6mm, VIA'S:VIA_0.6mm, F.Cu at (169.8, 85.8)
- added REF**: VIA_0.6mm, VIA'S:VIA_0.6mm, F.Cu at (169.8, 80.8)
- added REF**: VIA_0.6mm, VIA'S:VIA_0.6mm, F.Cu at (169.8, 75.8)
- added REF**: VIA_0.6mm, VIA'S:VIA_0.6mm, F.Cu at (163.4, 105.8)
- added REF**: VIA_0.6mm, VIA'S:VIA_0.6mm, F.Cu at (134.8, 70.8)
- added REF**: VIA_0.6mm, VIA'S:VIA_0.6mm, F.Cu at (144.8, 70.8)
- added REF**: VIA_0.6mm, VIA'S:VIA_0.6mm, F.Cu at (164.8, 70.8)
- added REF**: VIA_0.6mm, VIA'S:VIA_0.6mm, F.Cu at (159.8, 70.8)
- added REF**: VIA_0.6mm, VIA'S:VIA_0.6mm, F.Cu at (154.8, 70.8)
- added REF**: VIA_0.6mm, VIA'S:VIA_0.6mm, F.Cu at (157.9, 100.9)
- added REF**: VIA_0.6mm, VIA'S:VIA_0.6mm, F.Cu at (153.4, 101.0)
- added REF**: VIA_0.6mm, VIA'S:VIA_0.6mm, F.Cu at (128.5, 121.5)
- added REF**: VIA_0.6mm, VIA'S:VIA_0.6mm, F.Cu at (158.6, 113.4)
- added REF**: VIA_0.6mm, VIA'S:VIA_0.6mm, F.Cu at (137.7, 100.8)
- added REF**: VIA_0.6mm, VIA'S:VIA_0.6mm, F.Cu at (170.9, 115.4)
- added REF**: VIA_0.6mm, VIA'S:VIA_0.6mm, F.Cu at (167.4, 115.4)
- added REF**: VIA_0.6mm, VIA'S:VIA_0.6mm, F.Cu at (163.3, 116.3)
- added REF**: VIA_0.6mm, VIA'S:VIA_0.6mm, F.Cu at (158.6, 110.6)
- added REF**: VIA_0.6mm, VIA'S:VIA_0.6mm, F.Cu at (142.6, 111.7)
- added REF**: VIA_0.6mm, VIA'S:VIA_0.6mm, F.Cu at (139.3, 111.7)
- added REF**: VIA_0.6mm, VIA'S:VIA_0.6mm, F.Cu at (140.5, 121.5)
- added REF**: VIA_0.6mm, VIA'S:VIA_0.6mm, F.Cu at (143.6, 121.5)
- added REF**: VIA_0.6mm, VIA'S:VIA_0.6mm, F.Cu at (137.7, 116.5)
- added REF**: VIA_0.6mm, VIA'S:VIA_0.6mm, F.Cu at (139.9, 114.6)
- added REF**: VIA_0.6mm, VIA'S:VIA_0.6mm, F.Cu at (132.7, 100.8)
- added REF**: VIA_0.6mm, VIA'S:VIA_0.6mm, F.Cu at (150.2, 114.4)
- added REF**: VAL**, conn-wire-pads:Hole-Screw-NP-#2, F.Cu at (128.2, 100.5)
- added REF**: VIA_0.6mm, VIA'S:VIA_0.6mm, F.Cu at (149.8, 90.8)
- added REF**: VAL**, conn-wire-pads:Hole-Screw-NP-#2, F.Cu at (169.7, 100.5)
- added REF**: VAL**, conn-wire-pads:Hole-Screw-NP-#2, F.Cu at (169.7, 71.6)
- added REF**: VIA_0.6mm, VIA'S:VIA_0.6mm, F.Cu at (149.8, 85.8)
- added REF**: VIA_0.6mm, VIA'S:VIA_0.6mm, F.Cu at (149.8, 80.8)
- added REF**: VIA_0.6mm, VIA'S:VIA_0.6mm, F.Cu at (149.8, 75.8)
- added REF**: VIA_0.6mm, VIA'S:VIA_0.6mm, F.Cu at (127.7, 95.8)
- P1: value MICRO_USB -> Micro_usb_B
- U2: footprint Housings_DFN_QFN:QFN-28-1EP_5x5mm_Pitch0.5mm -> smt-dfn:QFN-28-1EP_5x5mm_Pitch0.5mm
- moved U3 11.6 mm to (136.9, 114.0)
- moved R3 11.0 mm to (136.5, 118.3)
- moved D3 10.9 mm to (141.0, 118.3)
- moved P2 10.1 mm to (129.4, 104.5)
- moved REF** 9.86 mm to (77.6, 69.6)
- moved C1 9.77 mm to (155.9, 108.1)
- moved C3 9.53 mm to (132.5, 119.0)
- moved C4 9.53 mm to (132.5, 113.8)
- moved C5 9.53 mm to (153.2, 113.8)
- moved C6 9.53 mm to (144.8, 113.4)
- moved D1 9.53 mm to (142.7, 110.0)
- moved G*** 9.53 mm to (149.1, 98.6)
- moved P1 9.53 mm to (149.0, 120.0)
- moved P3 9.53 mm to (133.0, 75.0)
- moved P4 9.53 mm to (169.3, 118.0)
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Connections:
- P2 pad 1: GND -> Net-(P2-Pad1)
- P2 pad 2: Net-(P2-Pad2) -> GND
- SW1 pad 1: Net-(P2-Pad2) -> Net-(P2-Pad1)
Routing:
- net GND: track 45.9 -> 28.3 mm
- net Net-(P2-Pad1): track 0.00 -> 14.1 mm
- net Net-(P2-Pad2): track 6.77 -> 0.00 mm
- net VXBEE_3V3: track 83.9 -> 87.2 mm
- net Net-(C3-Pad1): track 8.85 -> 11.1 mm
- net +5V: track 46.7 -> 48.6 mm, vias 0 -> 2
Other:
- board size 45 x 53 mm -> 45.5 x 53 mm
- rule trace_min: 0.2 -> 0.15
- rule via_min_drill: 0.3 -> 0.25
- rule via_min_size: 0.4 -> 0.25
- board text added: "53 x 45.5"
- board text added: "BOT"
- board text added: "RTS/DIO6"
- board text added: "TOP"
- board text added: "XBee Socket"
- board text removed: "53 x 45"
- board text removed: "RTS/A6/IO6"

Commit message: version of board added in silkscreen
Other:
- board text added: "v1.0"
Changed lines of the file:
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@@
     (area 126.199999 69.549999 171.800001 122.650001)
     (thickness 1.6)
-    (drawings 45)
+    (drawings 46)
     (tracks 299)
     (zones 0)
@@
       (clearance 0.5) (zone_connect 0))
   )
+  (gr_text v1.0 (at 137.34 103.5) (layer B.SilkS)
+    (effects (font (size 1.5 1.5) (thickness 0.3)) (justify mirror))
+  )
   (dimension 45.501758 (width 0.3) (layer Dwgs.User)
